File: pcb/plant_sensor.kicad_pcb (KiCad board)
At the start: 2 copper layers, 23 parts, among them IC1 SPBTLE-RF0, IC2 STM32L052K8Tx, J1 Conn_ARM_JTAG_SWD_10, J2 COM, U1 M95256-WMN6P, U2 LM75B, Y1 32.768kHz

Commit message: WIP
Parts:
- added R6: 4K7, Resistors_SMD:R_0805_HandSoldering, F.Cu at (43.9, 87.8)
- added R7: 4K7, Resistors_SMD:R_0805_HandSoldering, F.Cu at (43.9, 89.7)
- added R8: 10K, Resistors_SMD:R_0805_HandSoldering, F.Cu at (51.8, 87.8)
- added SW1: SW_Push, Buttons_Switches_SMD:SW_SPST_SKQG, F.Cu at (37.3, 89.8)
- BT1: moved to B.Cu
- Y1: footprint Crystals:Crystal_SMD_HC49-SD_HandSoldering -> Crystals:Crystal_SMD_TXC_9HT11-2pin_2.0x1.2mm_HandSoldering
- moved BT1 144.5 mm to (226.6, 79.8)
- moved Y1 3.07 mm to (146.6, 77.7)
