File: pcb/plant-sensor.brd (EAGLE design)
At the start: 160 x 100 mm, 40 parts, among them IC1 MCP73831/OT, IC17 LD398533RM, IC3 STM32L052K8T, U14 PCT2075D, U5 SPBTLE-RF, X1 JTAG, Y2 32.768kHz

Commit message: layouting
Parts:
- removed C47, C56, C62: 100nF, resistor:C0805
- removed C49: 10uF, resistor:C0805
- removed C57: 10nF X7R, resistor:C0805
- removed C58, C61: 1uF_X5R, resistor:C0805
- removed D13: BAT60JFILM, diode:SOD323-W
- removed IC17: LD398533RM, st-microelectronics:SOT23-5L
- removed LED3: RED, led:CHIP-LED0805
- removed R15: 10K, resistor:R0805
- removed U14: PCT2075D, clock:SOIC8_150MIL
- removed U5: SPBTLE-RF, clock:XCVR_SPBTLE-RF
- removed Y2: 32.768kHz, clock:XTAL_ABS25-32.768KHZ-6-1-T
- added C17, C3, C7: 100nF, resistor:C0805
- added C18: 10uF, resistor:C0805
- added C19: 10nF, resistor:C0805
- added C20: 1nF, resistor:C0805
- added C21: 47pF, resistor:C0805
- added C4: 10nF X7R, resistor:C0805
- added C5: 4.7uF, resistor:C0805
- added C6: 1uF_X5R, resistor:C0805
- added C8: 3pF, resistor:C0805
- added C9: 1uF, resistor:C0805
- added CN1: (no value), adafruit:JST-PH-2-SMT-RA
- added D1: BAT60JFILM, diode:SOD323-W
- added D2: PMEG6020AELRX, diode:SOD123
- added D3: USBLC6-2SC6, clock:SOT95P280X145-6N
- added F1, F2: MF-PSMF050X-2MF-PSMF, custom:R0805
- added IC2: LD398533RM, st-microelectronics:SOT23-5L
- added LED2: RED, led:CHIP-LED0805
- added Q1: IRLML6402, transistor-power:MICRO3
- added R1: 2K, resistor:R0805
- added R11: 10K, resistor:R0805
- added R12, R13: 15R, resistor:R0805
- added U1: PCT2075D, custom:SOIC8_150MIL
- added U2: SPBTLE-RF, custom:XCVR_SPBTLE-RF
- added X2: USB-MICROB, custom:USB-MICROB
- added Y1: 32.768kHz, custom:XTAL_ABS25-32.768KHZ-6-1-T
- C1: value 1uF_X5R -> 4.7uF
- C10: value 1uF -> 3pF
- C11, C13: value 3pF -> 100nF
- C16: value 100nF -> 10uF
- C22: value 100nF -> 1nF
- C23: value 10uF -> 47pF
- R10, R9: value 100K -> 2K2
- R4, R5: value 10K -> 100K
- R6: value 1K -> 10K
- R7: value 2K2 -> 10K
- R8: value 2K2 -> 1K
- S1: device clock:B3S-10XX -> custom:B3S-10XX
- moved C2 247.2 mm to (123.2, 34.9)
- moved R3 208.0 mm to (54.3, 30.5), turned to 180 degrees
- moved C1 203.6 mm to (49.8, 33.7), turned to 270 degrees
- moved R10 190.9 mm to (-2.86, 4.13), turned to 270 degrees
- moved R2 185.1 mm to (50.8, 26.7), turned to 180 degrees
- moved R9 184.5 mm to (-5.08, 4.13), turned to 270 degrees
- moved LED1 129.3 mm to (50.5, 24.4), turned to 90 degrees
- moved C13 120.5 mm to (-5.08, 17.8), turned to 180 degrees
- moved L1 116.8 mm to (8.57, 13.7), turned to 270 degrees
- moved C11 115.7 mm to (6.35, 13.7), turned to 270 degrees
- moved R7 112.0 mm to (10.8, 13.7), turned to 90 degrees
- moved C15 111.5 mm to (3.81, 19.7), turned to 180 degrees
- moved X1 111.3 mm to (-25.1, 18.4), turned to 90 degrees
- moved R8 111.1 mm to (13.0, 8.89), turned to 90 degrees
- moved C16 111.0 mm to (3.81, 17.5), turned to 180 degrees
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Connections:
- new net N$107: D3.1, X2.D-
- new net N$108: D3.4, R12.1
- new net N$2: CN1.1, F1.1
- new net N$22: D3.6, R13.1
- new net N$3: C2.1, C3.1, D1.C, IC2.1, IC2.3, Q1.2
- new net N$6: C20.1, D3.5, F2.2, X2.VBUS
- new net N$7: D3.3, X2.D+
- new net N$8: C19.1, X2.MT1, X2.MT2
- net !RESET: now also C12.2, R7.1; no longer C14.2, R5.1
- net !SPI_BLE_RESET: now also U2.11; no longer U5.11
- net +3V3: now also C13.2, C14.2, C15.1, C16.1, C17.1, C18.2, C6.1, C7.1, IC2.5, R10.2, R11.2, R9.2, U1.8, U2.5; no longer C15.2, C16.2, C22.1, C23.2, C47.1, C49.1, C61.1, C62.1, IC17.5, R15.2, R5.2, R8.2, U14.8, U5.5
- net BOOT0: now also R6.2; no longer R4.2
- net CHARGE: now also IC3.8, LED1.C; no longer IC3.7, LED3.C
- net GND: now also C10.2, C11.1, C13.1, C15.2, C16.2, C17.2, C18.1, C19.2, C20.2, C21.2, C23.2, C3.2, C4.2, C5.2, C6.2, C7.2, C8.2, C9.1, CN1.2, D2.A, D3.2, IC2.2, LED2.C, R1.1, R5.1, R6.1, U1.4, U1.5, U1.6, U1.7, U2.6, X2.GND; no longer C10.1, C11.2, C13.2, C15.1, C16.1, C23.1, C47.2, C49.2, C56.2, C57.2, C58.2, C61.2, C62.2, IC17.2, LED1.C, R10.1, R4.1, U14.4, U14.5, U14.6, U14.7, U5.6
- net I2C2_SCL: now also R9.1, U1.2; no longer R7.1, U14.2
- net I2C2_SDA: now also R10.1, U1.1; no longer R8.1, U14.1
- net LED: now also IC3.6, R8.2; no longer IC3.10, R6.2
- net N$102: now also C4.1, IC2.4; no longer C57.1, IC17.4
- net N$4: now also LED1.A; no longer LED3.A
- net N$9: now also LED2.A, R8.1; no longer LED1.A, R6.1
- net RCC_OSC32_IN: now also C8.1, Y1.1; no longer C11.1, Y2.1
- net RCC_OSC32_OUT: now also C10.1, Y1.4; no longer C13.1, Y2.4
- net SPI_BLE_CS: now also U2.10; no longer U5.10
- net SPI_BLE_IRQ: now also R11.1, U2.4; no longer R15.1, U5.4
- net SPI_MISO: now also U2.8; no longer U5.8
- net SPI_MOSI: now also U2.9; no longer U5.9
- net SPI_SCK: now also U2.7; no longer U5.7
- net USB_D+: now also C21.1, R12.2
- net USB_D-: now also C23.1, R13.2
- net U_BAT: now also IC3.7, R4.1, R5.2; no longer IC3.6, R10.2, R9.1
- net VDDA: now also C11.2, C9.2; no longer C10.2, C12.2
- net V_BATT: now also C5.1, D2.C, F1.2, Q1.3, R4.2; no longer C2.1, D13.A, R9.2
- net V_USB: now also C22.1, D1.A, F2.1, Q1.1, R1.2; no longer C56.1, C58.1, D13.C, IC17.1, IC17.3
Routing:
- net LED: track 0.00 -> 15.4 mm, vias 0 -> 2
- net !RESET: track 0.00 -> 12.7 mm
- net +3V3: track 0.00 -> 12.6 mm
- net RCC_OSC32_OUT: track 0.00 -> 10.6 mm
- net N$6: track 0.00 -> 9.57 mm
- net RCC_OSC32_IN: track 0.00 -> 8.19 mm
- net VDDA: track 0.00 -> 7.61 mm
- net SPI_BLE_CS: track 0.00 -> 4.34 mm, vias 0 -> 1
- net SPI_MISO: track 0.00 -> 3.89 mm, vias 0 -> 1
- net SPI_MOSI: track 0.00 -> 3.83 mm, vias 0 -> 1
- net SPI_BLE_IRQ: track 0.00 -> 3.82 mm, vias 0 -> 1
- net SPI_SCK: track 0.00 -> 3.51 mm, vias 0 -> 1
- net I2C2_SCL: track 0.00 -> 2.92 mm, vias 0 -> 1
- net N$7: track 0.00 -> 2.79 mm
- net N$107: track 0.00 -> 2.78 mm
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- added copper zone on layer 1, net GND
- added copper zone on layer 16, net GND
Other:
- board size 160 x 100 mm -> 30 x 80 mm
