File: pcb/plant-sensor.sch (EAGLE design)
At the start: 40 parts, among them IC1 MCP73831/OT, IC17 LD398533RM, IC3 STM32L052K8T, U14 PCT2075D, U5 SPBTLE-RF, X1 JTAG, Y2 32.768kHz

Commit message: layouting
Parts:
- removed C47: 100nF, resistor:C-EUC0805
- removed C49: 10uF, resistor:C-EUC0805
- removed C58: 1uF_X5R, resistor:C-EUC0805
- removed D13: BAT60JFILM, diode:DIODE-SOD323-W
- removed LED3: RED, led:LEDCHIP-LED0805
- removed U14: PCT2075D, clock:PCT2075D
- removed U5: SPBTLE-RF, clock:SPBTLE-RF
- removed Y2: 32.768kHz, clock:ABS25-32.768KHZ-6-1-T
- added C17: 100nF, resistor:C-EUC0805
- added C18: 10uF, resistor:C-EUC0805
- added C19: 10nF, resistor:C-EUC0805
- added C20: 1nF, resistor:C-EUC0805
- added C21: 47pF, resistor:C-EUC0805
- added C5: 4.7uF, resistor:C-EUC0805
- added C8: 3pF, resistor:C-EUC0805
- added C9: 1uF, resistor:C-EUC0805
- added CN1: (no value), adafruit:JST_2PIN-SMT-RA
- added D1: BAT60JFILM, diode:DIODE-SOD323-W
- added D2: PMEG6020AELRX, diode:DIODE-SOD123
- added D3: USBLC6-2SC6, clock:USBLC6-2SC6
- added F1, F2: MF-PSMF050X-2MF-PSMF, custom:MF-PSMF050X-2MF-PSMF
- added LED2: RED, led:LEDCHIP-LED0805
- added Q1: IRLML6402, transistor-power:IRLML5203
- added R1: 2K, resistor:R-EU_R0805
- added R12, R13: 15R, resistor:R-EU_R0805
- added U1: PCT2075D, custom:PCT2075D
- added U2: SPBTLE-RF, custom:SPBTLE-RF
- added X2: USB-MICROB, custom:USB-MICROB
- added Y1: 32.768kHz, custom:ABS25-32.768KHZ-6-1-T
- C1: value 1uF_X5R -> 4.7uF
- C10: value 1uF -> 3pF
- C11, C13: value 3pF -> 100nF
- C16: value 100nF -> 10uF
- C22: value 100nF -> 1nF
- C23: value 10uF -> 47pF
- R10, R9: value 100K -> 2K2
- R4, R5: value 10K -> 100K
- R6: value 1K -> 10K
- R7: value 2K2 -> 10K
- R8: value 2K2 -> 1K
- S1: device clock:B3S-10XX -> custom:B3S-10XX
- renumbered C56 to C3, C57 to C4, C61 to C6, C62 to C7, IC17 to IC2, R15 to R11
Connections:
- new net N$107: D3.I/O1_1, X2.D-
- new net N$108: D3.I/O2_2, R12.1
- new net N$2: CN1.2, F1.1
- new net N$22: D3.I/O1_2, R13.1
- new net N$3: C2.1, C3.1, D1.C, IC2.VIN, IC2.VINH, Q1.S
- new net N$6: C20.1, D3.VBUS, F2.2, X2.VBUS
- new net N$7: D3.I/O2_1, X2.D+
- new net N$8: C19.1, X2.MT
- net !RESET: now also C12.2, R7.1; no longer C14.2, R5.1
- net !SPI_BLE_RESET: now also U2.BT_RESET; no longer U5.BT_RESET
- net +3V3: now also C13.2, C14.2, C15.1, C16.1, C17.1, C18.2, R10.2, R9.2, U1.VCC, U2.VIN; no longer C15.2, C16.2, C22.1, C23.2, C47.1, C49.1, R5.2, R8.2, U14.VCC, U5.VIN
- net BOOT0: now also R6.2; no longer R4.2
- net CHARGE: now also IC3MCU.PA2, LED1.C; no longer IC3MCU.PA1, LED3.C
- net GND: now also C10.2, C11.1, C13.1, C15.2, C16.2, C17.2, C18.1, C19.2, C20.2, C21.2, C23.2, C5.2, C8.2, C9.1, CN1.1, D2.A, D3.GND, LED2.C, R1.1, R5.1, R6.1, U1.A0, U1.A1, U1.A2, U1.GND, U2.GND, X2.GND; no longer C10.1, C11.2, C13.2, C15.1, C16.1, C23.1, C47.2, C49.2, C58.2, LED1.C, R10.1, R4.1, U14.A0, U14.A1, U14.A2, U14.GND, U5.GND
- net I2C2_SCL: now also R9.1, U1.SCL; no longer R7.1, U14.SCL
- net I2C2_SDA: now also R10.1, U1.SDA; no longer R8.1, U14.SDA
- net LED: now also IC3MCU.PA0, R8.2; no longer IC3MCU.PA4, R6.2
- net N$4: now also LED1.A; no longer LED3.A
- net N$9: now also LED2.A, R8.1; no longer LED1.A, R6.1
- net RCC_OSC32_IN: now also C8.1, Y1.1; no longer C11.1, Y2.1
- net RCC_OSC32_OUT: now also C10.1, Y1.2; no longer C13.1, Y2.2
- net SPI_BLE_CS: now also U2.SPI_CS; no longer U5.SPI_CS
- net SPI_BLE_IRQ: now also U2.SPI_IRQ; no longer U5.SPI_IRQ
- net SPI_MISO: now also U2.SPI_MISO; no longer U5.SPI_MISO
- net SPI_MOSI: now also U2.SPI_MOSI; no longer U5.SPI_MOSI
- net SPI_SCK: now also U2.SPI_CLK; no longer U5.SPI_CLK
- net USB_D+: now also C21.1, R12.2
- net USB_D-: now also C23.1, R13.2
- net U_BAT: now also IC3MCU.PA1, R4.1, R5.2; no longer IC3MCU.PA0, R10.2, R9.1
- net VDDA: now also C11.2, C9.2; no longer C10.2, C12.2
- net V_BATT: now also C5.1, D2.C, F1.2, Q1.D, R4.2; no longer C2.1, D13.A, R9.2
- net V_USB: now also C22.1, D1.A, F2.1, Q1.G, R1.2; no longer C3.1, C58.1, D13.C, IC2.VIN, IC2.VINH
